File: CanaryCap PCB/CanaryCap.kicad_pcb (KiCad board)
At the start: 2 copper layers, 125 x 35 mm, 6 parts, among them U1 ESP32-C6-MINI-1, U3 LM3940 3.3V-SOT223, U4 TPS82130

Commit message: We gotta figure out git ignore
Parts:
- moved U1 1.00 mm to (204.9, 55.0)
Changed lines of the file:
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@@
 	(footprint "RF_Module:ESP32-C6-MINI-1"
 		(layer "F.Cu")
-		(at 205.925 55 -90)
+		(at 204.925 55 -90)
 		(descr "2.4 GHz Wi-Fi, Bluetooth, Zigbee and Thread combo chip, external antenna, https://www.espressif.com/sites/default/files/documentation/esp32-c6-mini-1_mini-1u_datasheet_en.pdf")
 		(tags "2.4 GHz Wi-Fi Bluetooth Zigbee Thread external antenna espressif  16.6*13.2mm")
@@
 			(polygon
 				(pts
-					(xy 211.525 76.6) (xy 211.525 33.4) (xy 231.925 33.4) (xy 231.925 76.6)
+					(xy 210.525 76.6) (xy 210.525 33.4) (xy 230.925 33.4) (xy 230.925 76.6)
 				)
 			)

Commit message: Pushing for new MCU
Parts:
- removed U1: ESP32-C6-MINI-1, RF_Module:ESP32-C6-MINI-1

Commit message: Board progress
Parts:
- added C10: 10pF, Capacitor_SMD:C_0603_1608Metric_Pad1.08x0.95mm_HandSolder, F.Cu at (138.7, 50.9)
- added C11: 10pF, Capacitor_SMD:C_0603_1608Metric_Pad1.08x0.95mm_HandSolder, F.Cu at (138.7, 53.5)
- added C12: 0.1uF, Capacitor_SMD:C_0603_1608Metric_Pad1.08x0.95mm_HandSolder, F.Cu at (143.0, 40.9)
- added C13: 1uF, Capacitor_SMD:C_0603_1608Metric_Pad1.08x0.95mm_HandSolder, F.Cu at (143.0, 43.4)
- added C14: 10uF, Capacitor_SMD:C_0603_1608Metric_Pad1.08x0.95mm_HandSolder, F.Cu at (143.0, 45.9)
- added C15: 10uF, Capacitor_SMD:C_0603_1608Metric_Pad1.08x0.95mm_HandSolder, F.Cu at (143.0, 48.4)
- added C16: 0.1uF, Capacitor_SMD:C_0603_1608Metric_Pad1.08x0.95mm_HandSolder, F.Cu at (143.0, 50.9)
- added C17: 0.1uF, Capacitor_SMD:C_0603_1608Metric_Pad1.08x0.95mm_HandSolder, F.Cu at (143.0, 53.5)
- added C18: 10uF, Capacitor_SMD:C_0603_1608Metric_Pad1.08x0.95mm_HandSolder, F.Cu at (122.5, 53.5)
- added C19: 1uF, Capacitor_SMD:C_0603_1608Metric_Pad1.08x0.95mm_HandSolder, F.Cu at (147.4, 40.9)
- added C2: 10uF, Capacitor_SMD:C_0603_1608Metric_Pad1.08x0.95mm_HandSolder, F.Cu at (122.5, 43.4)
- added C3: 22uF, Capacitor_SMD:C_0603_1608Metric_Pad1.08x0.95mm_HandSolder, F.Cu at (122.5, 45.9)
- added C4: .47uF, Capacitor_SMD:C_0603_1608Metric_Pad1.08x0.95mm_HandSolder, F.Cu at (122.5, 48.4)
- added C5: 22uF, Capacitor_SMD:C_0603_1608Metric_Pad1.08x0.95mm_HandSolder, F.Cu at (122.5, 50.9)
- added C6: 0.1uF, Capacitor_SMD:C_0603_1608Metric_Pad1.08x0.95mm_HandSolder, F.Cu at (138.7, 40.9)
- added C7: 10uF, Capacitor_SMD:C_0603_1608Metric_Pad1.08x0.95mm_HandSolder, F.Cu at (138.7, 43.4)
- added C8: 1uF, Capacitor_SMD:C_0603_1608Metric_Pad1.08x0.95mm_HandSolder, F.Cu at (138.7, 45.9)
- added C9: 1uF, Capacitor_SMD:C_0603_1608Metric_Pad1.08x0.95mm_HandSolder, F.Cu at (138.7, 48.4)
- added D1: ESD9B3.3ST5G, Diode_SMD:D_SOD-923, F.Cu at (130.6, 48.9)
- added J1: USB_C_Receptacle_USB2.0_14P, Connector_USB:USB_C_Receptacle_XKB_U262-16XN-4BVC11, F.Cu at (146.7, 65.9)
- added L1: 2nH, Inductor_SMD:L_0603_1608Metric, F.Cu at (144.2, 56.0)
- added R10: 22, Resistor_SMD:R_0603_1608Metric_Pad0.98x0.95mm_HandSolder, F.Cu at (138.7, 69.4)
- added R3: 10k, Resistor_SMD:R_0603_1608Metric_Pad0.98x0.95mm_HandSolder, F.Cu at (147.4, 43.4)
- added R4: 10k, Resistor_SMD:R_0603_1608Metric_Pad0.98x0.95mm_HandSolder, F.Cu at (147.4, 45.9)
- added R5: 10k, Resistor_SMD:R_0603_1608Metric_Pad0.98x0.95mm_HandSolder, F.Cu at (147.4, 48.4)
- added R6: 5k, Resistor_SMD:R_0603_1608Metric_Pad0.98x0.95mm_HandSolder, F.Cu at (147.4, 50.9)
- added R7: 5.1k, Resistor_SMD:R_0603_1608Metric_Pad0.98x0.95mm_HandSolder, F.Cu at (138.7, 61.9)
- added R8: 5.1k, Resistor_SMD:R_0603_1608Metric_Pad0.98x0.95mm_HandSolder, F.Cu at (138.7, 64.4)
- added R9: 22, Resistor_SMD:R_0603_1608Metric_Pad0.98x0.95mm_HandSolder, F.Cu at (138.7, 66.9)
- added SW1: SW_MEC_5E, Button_Switch_SMD:SW_SPST_EVQP2_MiddlePushTravel_H2.5mm, F.Cu at (153.6, 42.2)
- added SW2: SW_MEC_5E, Button_Switch_SMD:SW_SPST_EVQP2_MiddlePushTravel_H2.5mm, F.Cu at (153.6, 47.2)
- added U1: ESP32-C6FH4, Package_DFN_QFN:QFN-32-1EP_5x5mm_P0.5mm_EP3.7x3.7mm, F.Cu at (153.2, 53.4)
- added XTAL1: FW4000044Q, Library:CRYSTAL4_FW4000044Q_DIO, F.Cu at (140.4, 56.7)
- moved R1 69.6 mm to (122.5, 56.0)
- moved R2 69.6 mm to (122.5, 58.5)
- moved C1 69.1 mm to (122.5, 40.9)
- moved U4 61.4 mm to (127.0, 50.2)
- moved U3 53.3 mm to (129.6, 43.9), turned to 0 degrees
