File: CanaryCap PCB/CanaryCap.kicad_pcb (KiCad board)
At the start: 2 copper layers, 66.2 x 30 mm, 66 parts, among them J1 USB_C_Receptacle_USB2.0_16P, J2 Impact Connector, J3 Gas Connector, J4 Battery Connector, Q1 NMOS, Q2 PMOS_Substrate, SW1 SW_MEC_5E, SW2 SW_MEC_5E, SW4 SW_MEC_5E, U1 LMZM23601V5, U2 LM3940 3.3V-SOT223, U3 ESP32-C6FH4, U4 ADXL343

Commit message: bruh bruh bruh
Parts:
- moved AE1 199.8 mm to (176.5, 163.5), turned to 180 degrees
- moved L4 199.1 mm to (184.3, 169.5), turned to 180 degrees
- moved C23 196.2 mm to (187.6, 169.5)
- moved R4 194.3 mm to (193.5, 182.4), turned to -90 degrees
- moved C1 193.7 mm to (161.5, 166.3)
- moved C10 193.7 mm to (193.6, 167.8)
- moved C11 193.7 mm to (203.1, 173.8)
- moved C12 193.7 mm to (192.0, 177.4)
- moved C13 193.7 mm to (192.0, 169.4)
- moved C14 193.7 mm to (200.9, 169.5)
- moved C15 193.7 mm to (192.0, 174.0)
- moved C16 193.7 mm to (186.8, 173.9)
- moved C17 193.7 mm to (188.6, 174.0)
- moved C18 193.7 mm to (185.1, 173.9)
- moved C19 193.7 mm to (164.2, 173.5)
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Routing:
- net GNDREF: track 59.8 -> 191.6 mm, vias 1 -> 7
- net +3.3V: track 33.1 -> 128.6 mm, vias 1 -> 6
- net Impact_IO: track 3.35 -> 37.6 mm, vias 0 -> 2
- net Net-(U3-CHIP_PU): track 3.33 -> 36.3 mm
- net +5V: track 28.0 -> 54.0 mm
- net Impact_CLK: track 2.83 -> 26.9 mm
- net GAS_IN: track 6.51 -> 28.3 mm, vias 1 -> 2
- net ANT_MICRO: track 0.00 -> 10.8 mm
- net Net-(Q2-G): track 1.17 -> 11.4 mm, vias 1 -> 2
- net VBUS: track 31.3 -> 38.5 mm
- net Net-(D2-A): track 0.00 -> 7.04 mm
- net ANT_OUT: track 0.00 -> 6.93 mm
- net Net-(U3-GPIO8): track 12.3 -> 8.52 mm
- net GAS_DIG_IN: track 27.6 -> 26.0 mm, vias 1 -> 2

Commit message: YIPPEE
Parts:
- removed AE1: WE-MCA_74889102450, Library:WE-MCA_74889102450
- removed C10, C9: 10pF, Capacitor_SMD:C_0603_1608Metric_Pad1.08x0.95mm_HandSolder
- removed C11, C12, C15, C16: 0.1uF, Capacitor_SMD:C_0603_1608Metric_Pad1.08x0.95mm_HandSolder
- removed C13, C14, C18: 10uF, Capacitor_SMD:C_0603_1608Metric_Pad1.08x0.95mm_HandSolder
- removed C17: 1uF, Capacitor_SMD:C_0603_1608Metric_Pad1.08x0.95mm_HandSolder
- removed C23: 1pF, Capacitor_SMD:C_0603_1608Metric_Pad1.08x0.95mm_HandSolder
- removed J2: Impact Connector, Connector_Molex:Molex_CLIK-Mate_502443-0670_1x06-1MP_P2.00mm_Vertical
- removed L1: 2nH, Inductor_SMD:L_0603_1608Metric
- removed L4: 2nh, Inductor_SMD:L_0603_1608Metric
- removed R4: 5k, Resistor_SMD:R_0603_1608Metric_Pad0.98x0.95mm_HandSolder
- removed XTAL1: FW4000044Q, Library:CRYSTAL4_FW4000044Q_DIO
- added J5: Conn_01x04_Pin, Connector_PinHeader_2.54mm:PinHeader_1x04_P2.54mm_Vertical, F.Cu at (222.5, 181.8)
- added LS1: AT-1440-TT-R, Library:XDCR_AT-1440-TT-R, F.Cu at (217.8, 165.0)
- added U5: H3LIS100DLTR, Library:H3LIS100DLTR, F.Cu at (215.3, 177.2)
- U3: value ESP32-C6FH4 -> ESP32-C6-WROOM-1-N8; footprint Package_DFN_QFN:QFN-32-1EP_5x5mm_P0.5mm_EP3.7x3.7mm -> Library:XCVR_ESP32-C6-WROOM-1-N8
- moved R10 10.3 mm to (212.8, 172.2)
- moved R9 10.3 mm to (212.8, 174.0)
- moved D4 7.43 mm to (175.9, 159.2)
- moved D8 7.43 mm to (186.3, 159.2)
- moved J3 7.43 mm to (194.1, 161.4)
- moved R18 7.43 mm to (181.1, 162.8)
- moved R19 7.43 mm to (183.7, 162.8)
- moved R20 7.43 mm to (186.3, 162.8)
- moved D5 7.43 mm to (178.5, 159.2)
- moved D6 7.43 mm to (181.1, 159.2)
- moved D7 7.43 mm to (183.7, 159.2)
- moved R16 7.43 mm to (175.9, 162.8)
- moved R17 7.43 mm to (178.5, 162.8)
- moved U4 7.06 mm to (215.4, 182.0)
- moved U3 5.64 mm to (198.5, 179.9), turned to 180 degrees
Connections:
- C8 pad 1: Net-(U3-CHIP_PU) -> Net-(U3-EN)
- R3 pad 2: Net-(U3-CHIP_PU) -> Net-(U3-EN)
- U3 pad 1: ANT_MICRO -> GNDREF
- U3 pad 10: GAS_IN -> BOOT
- U3 pad 12: unconnected-(U3-GPIO6/MTCK-Pad12) -> GAS_IN
- U3 pad 13: unconnected-(U3-GPIO7/MTDO-Pad13) -> USB_DN
- U3 pad 14: Net-(U3-GPIO8) -> USB_DP
- U3 pad 15: BOOT -> unconnected-(U3-IO9-Pad15)
- U3 pad 16: USB_DN -> unconnected-(U3-IO18-Pad16)
- U3 pad 17: USB_DP -> BUZZER
- U3 pad 18: Impact_IO -> HEARTBEAT
- U3 pad 19: Impact_CLK -> HEALTH
- U3 pad 2: Net-(U3-VDDA3P3) -> +3.3V
- U3 pad 20: +3.3V -> STATUS
- U3 pad 21: unconnected-(U3-U0TXD/GPIO16-Pad21) -> PENDING
- U3 pad 23: HEARTBEAT -> CANCEL
- U3 pad 24: HEALTH -> unconnected-(U3-RXD0/GPIO17-Pad24)
- U3 pad 25: STATUS -> unconnected-(U3-TXD0/GPIO16-Pad25)
- U3 pad 26: PENDING -> unconnected-(U3-IO3-Pad26)
- U3 pad 28: unconnected-(U3-SDIO_DATA3/GPIO23-Pad28) -> GNDREF
- U3 pad 3: Net-(U3-VDDA3P3) -> Net-(U3-EN)
- U3 pad 4: Net-(U3-CHIP_PU) -> TMS
- U3 pad 5: +3.3V -> TDI
- U3 pad 6: unconnected-(U3-GPIO0/XTAL_32K_P-Pad6) -> TCK
- U3 pad 7: unconnected-(U3-GPIO1/XTAL_32K_N-Pad7) -> TDO
- U3 pad 8: unconnected-(U3-GPIO2-Pad8) -> Impact_IO
- U3 pad 9: CANCEL -> Impact_CLK
Routing:
- net Net-(U3-EN): track 0.00 -> 47.7 mm, vias 0 -> 2
- net Net-(U3-CHIP_PU): track 36.3 -> 0.00 mm, vias 1 -> 0
- net BUZZER: track 0.00 -> 31.2 mm, vias 0 -> 1
- net Impact_IO: track 37.6 -> 17.6 mm, vias 2 -> 0
- net TMS: track 0.00 -> 18.7 mm
- net USB_DP: track 40.0 -> 56.9 mm
- net GNDREF: track 191.6 -> 208.4 mm, vias 7 -> 4
- net TDO: track 0.00 -> 16.6 mm, vias 0 -> 1
- net TCK: track 0.00 -> 16.2 mm, vias 0 -> 1
- net TDI: track 0.00 -> 15.9 mm, vias 0 -> 1
- net Impact_CLK: track 26.9 -> 11.0 mm
- net +3.3V: track 128.6 -> 112.7 mm, vias 6 -> 0
- net BOOT: track 35.9 -> 51.5 mm
- net GAS_IN: track 28.3 -> 16.1 mm, vias 2 -> 0
- net USB_DN: track 42.0 -> 53.5 mm
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Other:
- board size 66.2 x 30 mm -> 76 x 30 mm

Commit message: Bruh
Parts:
- added G***: LOGO, Library:canary, F.Cu at (148.2, 103.2)
- added G***: LOGO, Library:canary, B.Cu at (123.0, 101.2)
- added J2: Conn_02x04_Counter_Clockwise, Connector_Harwin:Harwin_LTek-Male_2x04_P2.00mm_Vertical, F.Cu at (153.8, 92.2)
- moved D5 86.5 mm to (127.0, 89.8)
- moved D6 86.5 mm to (129.6, 89.8)
- moved D7 86.5 mm to (132.2, 89.8)
- moved J5 86.5 mm to (170.9, 112.4)
- moved R10 86.5 mm to (161.3, 102.8)
- moved R15 86.5 mm to (133.1, 112.0)
- moved R16 86.5 mm to (124.3, 93.4)
- moved R17 86.5 mm to (126.9, 93.4)
- moved R9 86.5 mm to (161.3, 104.5)
- moved SW4 86.5 mm to (129.5, 114.9)
- moved U1 86.5 mm to (113.1, 97.3)
- moved U3 86.5 mm to (146.9, 110.5)
- moved U4 86.5 mm to (163.8, 112.5)
- moved U5 86.5 mm to (163.7, 107.8)
- moved C1 86.5 mm to (110.0, 96.8)
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Connections:
- U3 pad 30_10: GNDREF -> (no net)
- U3 pad 30_11: GNDREF -> (no net)
- U3 pad 30_12: GNDREF -> (no net)
- U3 pad 30_2: GNDREF -> (no net)
- U3 pad 30_8: GNDREF -> (no net)
- U3 pad 30_9: GNDREF -> (no net)
Routing:
- net STATUS: track 15.5 -> 45.1 mm
- net HEALTH: track 15.7 -> 43.7 mm, vias 2 -> 3
- net HEARTBEAT: track 16.2 -> 44.1 mm, vias 2 -> 3
- net +3.3V: track 112.7 -> 136.5 mm, vias 0 -> 2
- net PENDING: track 15.2 -> 38.9 mm
- net Impact_CLK: track 11.0 -> 27.0 mm, vias 0 -> 3
- net GNDREF: track 208.4 -> 215.1 mm, vias 4 -> 6
- net BUZZER: track 31.2 -> 37.7 mm
- net Impact_IO: track 17.6 -> 21.7 mm
- net TMS: track 18.7 -> 17.4 mm, vias 0 -> 1
- net Net-(U3-EN): track 47.7 -> 47.2 mm
Other:
- board size 76 x 30 mm -> 80 x 30 mm
- board text added: "CanaryCap"
- board text added: "Sebastian Arthur Vinny O'Byrne Justin Betz Elise Bauerschmidt"

Commit message: Capcb updates
Parts:
- J2: footprint Connector_Harwin:Harwin_LTek-Male_2x04_P2.00mm_Vertical -> Connector_PinHeader_2.54mm:PinHeader_2x04_P2.54mm_Vertical
- J3: value Gas Connector -> Conn_01x04_Pin; footprint Connector_Molex:Molex_CLIK-Mate_502443-0470_1x04-1MP_P2.00mm_Vertical -> Connector_PinHeader_2.54mm:PinHeader_1x04_P2.54mm_Vertical
- J4: value Battery Connector -> Conn_01x02_Pin; footprint Connector_Molex:Molex_CLIK-Mate_502443-0270_1x02-1MP_P2.00mm_Vertical -> Connector_PinHeader_2.54mm:PinHeader_1x02_P2.54mm_Vertical
- U2: value LM3940 3.3V-SOT223 -> NCP1117-3.3_SOT223
- moved J3 3.30 mm to (139.9, 90.0), turned to 90 degrees
- moved J4 2.78 mm to (100.5, 109.0), turned to 0 degrees
- moved U4 0.60 mm to (163.2, 112.5), turned to 90 degrees
- moved J2 0.29 mm to (153.5, 92.2), turned to 90 degrees
Connections:
- J3 pad 2: GAS_DIG_IN -> GNDREF
- J3 pad 3: GAS_IN -> GAS_DIG_IN
- J3 pad 4: GNDREF -> GAS_IN
- U3 pad 11: GAS_DIG_IN -> Impact_IO
- U3 pad 12: GAS_IN -> Impact_CLK
- U3 pad 16: unconnected-(U3-IO18-Pad16) -> BUZZER
- U3 pad 17: BUZZER -> HEARTBEAT
- U3 pad 18: HEARTBEAT -> HEALTH
- U3 pad 19: HEALTH -> STATUS
- U3 pad 20: STATUS -> PENDING
- U3 pad 21: PENDING -> CANCEL
- U3 pad 23: CANCEL -> unconnected-(U3-IO15-Pad23)
- U3 pad 26: unconnected-(U3-IO3-Pad26) -> GAS_IN
- U3 pad 27: unconnected-(U3-IO2-Pad27) -> GAS_DIG_IN
- U3 pad 30_1: (no net) -> GNDREF
- U3 pad 30_10: (no net) -> GNDREF
- U3 pad 30_11: (no net) -> GNDREF
- U3 pad 30_12: (no net) -> GNDREF
- U3 pad 30_2: (no net) -> GNDREF
- U3 pad 30_3: (no net) -> GNDREF
- U3 pad 30_4: (no net) -> GNDREF
- U3 pad 30_5: (no net) -> GNDREF
- U3 pad 30_6: (no net) -> GNDREF
- U3 pad 30_7: (no net) -> GNDREF
- U3 pad 30_8: (no net) -> GNDREF
- U3 pad 30_9: (no net) -> GNDREF
- U3 pad 8: Impact_IO -> unconnected-(U3-IO0-Pad8)
- U3 pad 9: Impact_CLK -> unconnected-(U3-IO1-Pad9)
- U4 pad 12: unconnected-(U4-SDO/ADDR-Pad12) -> GNDREF
- U4 pad 6: unconnected-(U4-Vs-Pad6) -> +3.3V
- U4 pad 7: unconnected-(U4-~{CS}-Pad7) -> +3.3V
- U5 pad 4: Impact_IO -> Impact_CLK
- U5 pad 6: Impact_CLK -> Impact_IO
- U5 pad 7: unconnected-(U5-SDO/SA0-Pad7) -> GNDREF
- U5 pad 8: unconnected-(U5-CS-Pad8) -> +3.3V
Routing:
- net +3.3V: track 136.5 -> 119.2 mm
- net GAS_IN: track 16.1 -> 28.7 mm, vias 0 -> 1
- net GAS_DIG_IN: track 18.6 -> 30.9 mm, vias 0 -> 1
- net +12V: track 19.9 -> 30.6 mm
- net Impact_CLK: track 27.0 -> 17.1 mm, vias 3 -> 0
- net USB_DP: track 56.7 -> 48.4 mm
- net BUZZER: track 37.7 -> 31.3 mm, vias 1 -> 2
- net GNDREF: track 215.1 -> 209.3 mm, vias 6 -> 11
- net STATUS: track 45.1 -> 39.4 mm, vias 2 -> 3
- net HEARTBEAT: track 44.1 -> 48.8 mm, vias 3 -> 1
- net PENDING: track 38.9 -> 35.0 mm
- net +5V: track 46.6 -> 50.2 mm
- net TMS: track 17.4 -> 20.9 mm
- net USB_DN: track 53.4 -> 50.4 mm
- net TDI: track 15.8 -> 18.6 mm
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