File: CanaryCap PCB/io.kicad_sch (KiCad schematic)
At the start: 5 parts, among them J1 USB_C_Receptacle_USB2.0_14P

Commit message: Updated schematics for justin to work
Parts:
- added C25: 22uF, Capacitor_SMD:C_0603_1608Metric_Pad1.08x0.95mm_HandSolder, symbol Device:C
- added D2: BZV55C5V6, Diode_SMD:D_MiniMELF, symbol Diode:BZV55C5V6
- added R15: 2.2k, Resistor_SMD:R_0603_1608Metric_Pad0.98x0.95mm_HandSolder, symbol Device:R_Small
- added R17: 100k, Resistor_SMD:R_0603_1608Metric_Pad0.98x0.95mm_HandSolder, symbol Device:R_Small
- added R19: 100, Resistor_SMD:R_0603_1608Metric_Pad0.98x0.95mm_HandSolder, symbol Device:R_Small
- J1: value USB_C_Receptacle_USB2.0_14P -> USB_C_Receptacle_USB2.0_16P; footprint Connector_USB:USB_C_Receptacle_XKB_U262-16XN-4BVC11 -> Connector_USB:USB_C_Receptacle_G-Switch_GT-USB-7010ASV
- renumbered R8 to R10, R9 to R7, R10 to R8, R7 to R9
Connections:
- net GNDREF: now also R15.2
- net VBUS renamed +5V
- net +5V: now also C25.1, D2.1 (K), R17.1, R19.2
- new net: D2.2 (A), R15.1
- new net: C25.2, R17.2
Other:
- note added: "TODO: ADD MOSFET HERE>>"
- note added: "TODO: FIND AND ADD MOSFET HERE"
- moved on the sheet: R10, R7, R8, R9

Commit message: new changes
Parts:
- added J2: Conn_01x06_MountingPin, symbol Connector_Generic_MountingPin:Conn_01x06_MountingPin
- added J3: Conn_01x04_MountingPin, symbol Connector_Generic_MountingPin:Conn_01x04_MountingPin
- added R11, R13: 2.2k, Resistor_SMD:R_0603_1608Metric_Pad0.98x0.95mm_HandSolder, symbol Device:R_Small
- added U5: ADXL343, Package_LGA:LGA-14_3x5mm_P0.8mm_LayoutBorder1x6y, symbol Sensor_Motion:ADXL343
Connections:
- net +5V: now also J3.1 (Pin_1)
- net GNDREF: now also J2.6 (Pin_6), J3.4 (Pin_4), U5.2 (GND), U5.4 (GND), U5.5 (GND)
- new net +3.3V: J2.1 (Pin_1), R11.1, R13.1, U5.1 (Vdd_I/O)
- new net GAS_DIG_IN: J3.2 (Pin_2)
- new net GAS_IN: J3.3 (Pin_3)
- new net Impact_CLK: J2.4 (Pin_4), R13.2, U5.14 (SCL/SCLK)
- new net Impact_IO: J2.2 (Pin_2), R11.2, U5.13 (SDA/SDI/SDIO)
Other:
- note added: "GAS SENSOR CONNECTOR"
- note added: "IMPACT SENSOR CONNECTOR"
