File: CanaryCap PCB/power.kicad_sch (KiCad schematic)
At the start: 11 parts, among them U3 LM3940 3.3V-SOT223, U4 TPS82130

Commit message: Updated schematics for justin to work
Parts:
- renumbered C2 to C1, C1 to C2, C18 to C6, U4 to U1, U3 to U2
Connections:
- net +5V: no longer C3.1, R1.1, U1.4 (VOUT), U1.5 (VOUT)
- new net +5V_buck: C3.1, R1.1, U1.4 (VOUT), U1.5 (VOUT)
Changed lines of the file:
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@@
 		(dnp no)
 		(fields_autoplaced yes)
-		(property "Reference" "#PWR07"
+		(property "Reference" "#PWR08"
 			(at 157.48 85.09 0)
 			(effects
@@
 			(project "CanaryCap"
 				(path "/406ad30e-b04c-4bb7-9588-aab8ab73084a/3219e357-ed27-4a99-8f08-f1a850fa8309"
-					(reference "#PWR07")
+					(reference "#PWR08")
 					(unit 1)
 				)
@@
 		(dnp no)
 		(fields_autoplaced yes)
-		(property "Reference" "#PWR03"
+		(property "Reference" "#PWR01"
 			(at 66.04 83.82 0)
 			(effects
@@
 			(project "CanaryCap"
 				(path "/406ad30e-b04c-4bb7-9588-aab8ab73084a/3219e357-ed27-4a99-8f08-f1a850fa8309"
-					(reference "#PWR03")
+					(reference "#PWR01")
 					(unit 1)
 				)
@@
 		(dnp no)
 		(fields_autoplaced yes)
-		(property "Reference" "C2"
+		(property "Reference" "C1"
 			(at 71.12 82.5499 0)
 			(effects
@@
 			(project "CanaryCap"
 				(path "/406ad30e-b04c-4bb7-9588-aab8ab73084a/3219e357-ed27-4a99-8f08-f1a850fa8309"
-					(reference "C2")
+					(reference "C1")
 					(unit 1)
 				)
@@
 		(dnp no)
 		(fields_autoplaced yes)
-		(property "Reference" "U4"
+		(property "Reference" "U1"
 			(at 86.36 72.39 0)
 			(effects
@@
 			(project "CanaryCap"
 				(path "/406ad30e-b04c-4bb7-9588-aab8ab73084a/3219e357-ed27-4a99-8f08-f1a850fa8309"
-					(reference "U4")
+					(reference "U1")
 					(unit 1)
 				)
@@
 		(dnp no)
 		(fields_autoplaced yes)
-		(property "Reference" "#PWR010"
+		(property "Reference" "#PWR04"
 			(at 110.49 93.98 0)
 			(effects
@@
 			(project "CanaryCap"
 				(path "/406ad30e-b04c-4bb7-9588-aab8ab73084a/3219e357-ed27-4a99-8f08-f1a850fa8309"
-					(reference "#PWR010")
+					(reference "#PWR04")
 					(unit 1)
 				)
@@
 		(dnp no)
 		(fields_autoplaced yes)
-		(property "Reference" "#PWR04"
+		(property "Reference" "#PWR05"
 			(at 111.76 83.82 0)
 			(effects
@@
 			)
 		)
-		(property "Value" "+5V"
+		(property "Value" "+5V_buck"
 			(at 111.76 74.93 0)
 			(effects
@@
 			(project "CanaryCap"
 				(path "/406ad30e-b04c-4bb7-9588-aab8ab73084a/3219e357-ed27-4a99-8f08-f1a850fa8309"
-					(reference "#PWR04")
+					(reference "#PWR05")
 					(unit 1)
 				)
@@
 		(dnp no)
 		(fields_autoplaced yes)
-		(property "Reference" "#PWR019"
+		(property "Reference" "#PWR09"
 			(at 191.77 86.36 0)
 			(effects
@@
 			(project "CanaryCap"
 				(path "/406ad30e-b04c-4bb7-9588-aab8ab73084a/3219e357-ed27-4a99-8f08-f1a850fa8309"
-					(reference "#PWR019")
+					(reference "#PWR09")
 					(unit 1)
 				)
@@
 		(dnp no)
 		(fields_autoplaced yes)
-		(property "Reference" "#PWR05"
+		(property "Reference" "#PWR03"
 			(at 86.36 106.68 0)
 			(effects
@@
 			(project "CanaryCap"
 				(path "/406ad30e-b04c-4bb7-9588-aab8ab73084a/3219e357-ed27-4a99-8f08-f1a850fa8309"
-					(reference "#PWR05")
+					(reference "#PWR03")
 					(unit 1)
 				)
@@
 		(dnp no)
 		(fields_autoplaced yes)
-		(property "Reference" "C1"
+		(property "Reference" "C2"
 			(at 76.2 92.7099 0)
 			(effects
@@
 			(project "CanaryCap"
 				(path "/406ad30e-b04c-4bb7-9588-aab8ab73084a/3219e357-ed27-4a99-8f08-f1a850fa8309"
-					(reference "C1")
+					(reference "C2")
 					(unit 1)
 				)
@@
 		(on_board yes)
 		(dnp no)
-		(property "Reference" "C18"
+		(property "Reference" "C6"
 			(at 189.23 91.694 0)
 			(effects
@@
 			(project "CanaryCap"
 				(path "/406ad30e-b04c-4bb7-9588-aab8ab73084a/3219e357-ed27-4a99-8f08-f1a850fa8309"
-					(reference "C18")
+					(reference "C6")
 					(unit 1)
 				)
@@
 		(dnp no)
 		(fields_autoplaced yes)
-		(property "Reference" "#PWR020"
+		(property "Reference" "#PWR010"
 			(at 191.77 105.41 0)
 			(effects
@@
 			(project "CanaryCap"
 				(path "/406ad30e-b04c-4bb7-9588-aab8ab73084a/3219e357-ed27-4a99-8f08-f1a850fa8309"
-					(reference "#PWR020")
+					(reference "#PWR010")
 					(unit 1)
 				)
@@
 		(dnp no)
 		(fields_autoplaced yes)
-		(property "Reference" "U3"
+		(property "Reference" "U2"
 			(at 146.05 74.93 0)
 			(effects
@@
 			(project "CanaryCap"
 				(path "/406ad30e-b04c-4bb7-9588-aab8ab73084a/3219e357-ed27-4a99-8f08-f1a850fa8309"
-					(reference "U3")
+					(reference "U2")
 					(unit 1)
 				)
@@
 		(dnp no)
 		(fields_autoplaced yes)
-		(property "Reference" "#PWR08"
+		(property "Reference" "#PWR07"
 			(at 146.05 97.79 0)
 			(effects
@@
 			(project "CanaryCap"
 				(path "/406ad30e-b04c-4bb7-9588-aab8ab73084a/3219e357-ed27-4a99-8f08-f1a850fa8309"
-					(reference "#PWR08")
+					(reference "#PWR07")
 					(unit 1)
 				)
@@
 		(dnp no)
 		(fields_autoplaced yes)
-		(property "Reference" "#PWR09"
+		(property "Reference" "#PWR02"
 			(at 67.31 93.98 0)
 			(effects
@@
 			(project "CanaryCap"
 				(path "/406ad30e-b04c-4bb7-9588-aab8ab73084a/3219e357-ed27-4a99-8f08-f1a850fa8309"
-					(reference "#PWR09")
-					(unit 1)
-				)
+					(reference "#PWR02")
+					(unit 1)
+				)

Commit message: new changes
Parts:
- added C26, C27: 10uF, Capacitor_SMD:C_0603_1608Metric_Pad1.08x0.95mm_HandSolder, symbol Device:C
- added U4: LMZM23601V5, Package_LGA:Texas_SIL0010A_MicroSiP-10-1EP_3.8x3mm_P0.6mm_EP0.7x2.9mm_ThermalVias, symbol Regulator_Switching:LMZM23601V5
- C5: value 22uF -> 33uF
Connections:
- net +12V: now also C26.1, U4.3 (VIN), U4.4 (EN)
- net +5V_buck: now also C27.1, U4.6 (VOUT), U4.7 (FB)
- net GNDREF: now also C26.2, C27.2, U4.1 (GND), U4.11 (GND), U4.2 (MODE/SYNC)
- no-connect marks 0 -> 1
Other:
- note added: "This is what Elise has in her doc. Not sure why its depicted as a current output, maybe because it is controlled current"
