File: CanaryCap PCB/power.kicad_sch (KiCad schematic)
At the start: 8 parts, among them U1 LMZM23601V5, U2 LM3940 3.3V-SOT223

Commit message: Capcb updates
Parts:
- U2: value LM3940 3.3V-SOT223 -> NCP1117-3.3_SOT223
Changed lines of the file:
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@@
 			)
 		)
-		(property "Value" "LM3940 3.3V-SOT223"
+		(property "Value" "NCP1117-3.3_SOT223"
 			(at 146.05 77.47 0)
 			(effects
