File: CanaryCap PCB/CanaryCap.kicad_sch (KiCad schematic)
At the start: 0 parts

Commit message: We gotta figure out git ignore
Parts:
- added C1: C, Capacitor_SMD:C_0603_1608Metric_Pad1.08x0.95mm_HandSolder, symbol Device:C
- added C2, C6, C7, C8: 10uF, Capacitor_SMD:C_0603_1608Metric_Pad1.08x0.95mm_HandSolder, symbol Device:C
- added C3, C5: 22uF, Capacitor_SMD:C_0603_1608Metric_Pad1.08x0.95mm_HandSolder, symbol Device:C
- added C4: .47uF, Capacitor_SMD:C_0603_1608Metric_Pad1.08x0.95mm_HandSolder, symbol Device:C
- added C9: 1uF, Capacitor_SMD:C_0603_1608Metric_Pad1.08x0.95mm_HandSolder, symbol Device:C
- added R1: 540k, Resistor_SMD:R_0603_1608Metric_Pad0.98x0.95mm_HandSolder, symbol Device:R_Small
- added R2: 100k, Resistor_SMD:R_0603_1608Metric_Pad0.98x0.95mm_HandSolder, symbol Device:R_Small
- added R3: 10k, Resistor_SMD:R_0603_1608Metric_Pad0.98x0.95mm_HandSolder, symbol Device:R_Small
- added U1: ESP32-C6FH4, ESP32-C6FH4:QFN50P500X500X90-33N, symbol ESP-32-C6:ESP32-C6FH4
- added U3: LM3940 3.3V-SOT223, Package_TO_SOT_SMD:SOT-223-3_TabPin2, symbol Regulator_Linear:NCP1117-3.3_SOT223
- added U4: TPS82130, Package_LGA:Texas_SIL0008D_MicroSiP-8-1EP_2.8x3mm_P0.65mm_EP1.1x1.9mm_ThermalVias, symbol Regulator_Switching:TPS82130
Connections:
- new net: R1.2, R2.1, U4.6 (FB)
- new net: C1.1, U4.8 (SS/TR)
- new net: C9.1, R3.2, U1.4 (CHIP_PU)
- new net +12V: C2.1, U4.1 (EN), U4.2 (VIN)
- new net +3.3V: C5.1, C6.1, C7.1, C8.1, R3.1, U1.2 (VDDA3P3), U1.20 (VDDPST2), U1.29 (VDDA1), U1.3 (VDDA3P3__1), U1.32 (VDDA2), U1.5 (VDDPST1), U3.2 (VO)
- new net +5V: C3.1, C4.1, R1.1, U3.3 (VI), U4.4 (VOUT), U4.5 (VOUT)
- new net GNDREF: C1.2, C2.2, C3.2, C4.2, C5.2, C6.2, C7.2, C8.2, C9.2, R2.2, U1.33 (GND), U3.1 (GND), U4.3 (GND), U4.9 (GND)

Commit message: Pushing for new MCU
Parts:
- added Y1: Crystal_GND24, symbol Device:Crystal_GND24
Changed lines of the file:
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@@
+	)
+	(symbol
+		(lib_id "Device:Crystal_GND24")
+		(at 146.05 95.25 0)
+		(unit 1)
+		(exclude_from_sim no)
+		(in_bom yes)
+		(on_board yes)
+		(dnp no)
+		(fields_autoplaced yes)
+		(property "Reference" "Y1"
+			(at 157.48 88.8298 0)
+			(effects
+				(font
+					(size 1.27 1.27)
+				)
+			)
+		)
+		(property "Value" "Crystal_GND24"
+			(at 157.48 91.3698 0)
+			(effects
+				(font
+					(size 1.27 1.27)
+				)
+			)
+		)
+		(property "Footprint" ""
+			(at 146.05 95.25 0)
+			(effects
+				(font
+					(size 1.27 1.27)
+				)
+				(hide yes)
+			)
+		)
+		(property "Datasheet" "~"
+			(at 146.05 95.25 0)
+			(effects
+				(font
+					(size 1.27 1.27)
+				)
+				(hide yes)
+			)
+		)
+		(property "Description" "Four pin crystal, GND on pins 2 and 4"
+			(at 146.05 95.25 0)
+			(effects
+				(font
+					(size 1.27 1.27)
+				)
+				(hide yes)
+			)
+		)
+		(pin "4"
+		)
+		(pin "2"
+		)
+		(pin "1"
+		)
+		(pin "3"
+		)
+		(instances
+			(project ""
+				(path "/406ad30e-b04c-4bb7-9588-aab8ab73084a"
+					(reference "Y1")
+					(unit 1)
+				)
+			)
+		)
 	)
 	(symbol

Commit message: Board progress
Parts:
- removed C1: C, Capacitor_SMD:C_0603_1608Metric_Pad1.08x0.95mm_HandSolder, symbol Device:C
- removed C2, C6, C7, C8: 10uF, Capacitor_SMD:C_0603_1608Metric_Pad1.08x0.95mm_HandSolder, symbol Device:C
- removed C3, C5: 22uF, Capacitor_SMD:C_0603_1608Metric_Pad1.08x0.95mm_HandSolder, symbol Device:C
- removed C4: .47uF, Capacitor_SMD:C_0603_1608Metric_Pad1.08x0.95mm_HandSolder, symbol Device:C
- removed C9: 1uF, Capacitor_SMD:C_0603_1608Metric_Pad1.08x0.95mm_HandSolder, symbol Device:C
- removed R1: 540k, Resistor_SMD:R_0603_1608Metric_Pad0.98x0.95mm_HandSolder, symbol Device:R_Small
- removed R2: 100k, Resistor_SMD:R_0603_1608Metric_Pad0.98x0.95mm_HandSolder, symbol Device:R_Small
- removed R3: 10k, Resistor_SMD:R_0603_1608Metric_Pad0.98x0.95mm_HandSolder, symbol Device:R_Small
- removed U1: ESP32-C6FH4, ESP32-C6FH4:QFN50P500X500X90-33N, symbol ESP-32-C6:ESP32-C6FH4
- removed U3: LM3940 3.3V-SOT223, Package_TO_SOT_SMD:SOT-223-3_TabPin2, symbol Regulator_Linear:NCP1117-3.3_SOT223
- removed U4: TPS82130, Package_LGA:Texas_SIL0008D_MicroSiP-8-1EP_2.8x3mm_P0.65mm_EP1.1x1.9mm_ThermalVias, symbol Regulator_Switching:TPS82130
- removed Y1: Crystal_GND24, symbol Device:Crystal_GND24
Other:
- added sheet IO (io.kicad_sch)
- added sheet MicroConfig (micro.kicad_sch)
- added sheet Power_System (power.kicad_sch)

Commit message: Done with ts for the night
Other:
- sheet Power_System renamed PowerSystem
- title: (none) -> CanaryCapMain
Changed lines of the file:
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@@
 	(paper "A4")
 	(title_block
+		(title "CanaryCapMain")
 		(date "2025-10-01")
 	)
@@
 			(color 0 0 0 0.0000)
 		)
-		(property "Sheetname" "Power_System"
+		(property "Sheetname" "PowerSystem"
 			(at 26.67 41.1984 0)
 			(effects

Commit message: Updated schematics for justin to work
Other:
- added sheet RF (rf.kicad_sch)
Changed lines of the file:
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@@
+	)
+	(sheet
+		(at 105.41 100.33)
+		(size 66.04 41.91)
+		(exclude_from_sim no)
+		(in_bom yes)
+		(on_board yes)
+		(dnp no)
+		(fields_autoplaced yes)
+		(stroke
+			(width 0.1524)
+			(type solid)
+		)
+		(fill
+			(color 0 0 0 0.0000)
+		)
+		(property "Sheetname" "RF"
+			(at 105.41 99.6184 0)
+			(effects
+				(font
+					(size 1.27 1.27)
+				)
+				(justify left bottom)
+			)
+		)
+		(property "Sheetfile" "rf.kicad_sch"
+			(at 105.41 142.8246 0)
+			(effects
+				(font
+					(size 1.27 1.27)
+				)
+				(justify left top)
+			)
+		)
+		(instances
+			(project "CanaryCap"
+				(path "/406ad30e-b04c-4bb7-9588-aab8ab73084a"
+					(page "5")
+				)
+			)
+		)
 	)
 	(sheet

Commit message: Added todo
Other:
- note added: "TODO: Add piezo + a couple breakout pins on a connector just in case"
Changed lines of the file:
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@@
 		(date "2025-10-01")
+	)
+	(text "TODO: Add piezo + a couple breakout \npins on a connector just in case"
+		(exclude_from_sim no)
+		(at 209.042 53.086 0)
+		(effects
+			(font
+				(size 1.27 1.27)
+			)
+		)
 	)
 	(sheet

Commit message: FIXED IT MF
Other:
- note removed: "TODO: Add piezo + a couple breakout pins on a connector just in case"
Changed lines of the file:
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@@
 		(date "2025-10-01")
-	)
-	(text "TODO: Add piezo + a couple breakout \npins on a connector just in case"
-		(exclude_from_sim no)
-		(at 209.042 53.086 0)
-		(effects
-			(font
-				(size 1.27 1.27)
-			)
-		)
 	)
 	(sheet

Commit message: PCB layout started
Parts:
- added R12: 22, Resistor_SMD:R_0603_1608Metric_Pad0.98x0.95mm_HandSolder, symbol Device:R_Small
Connections:
- new net USB_DP: R12.1
Changed lines of the file:
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@@
 		(date "2025-10-01")
+	)
+	(wire
+		(pts
+			(xy 193.04 53.34) (xy 196.85 53.34)
+		)
+		(stroke
+			(width 0)
+			(type default)
+		)
+	)
+	(wire
+		(pts
+			(xy 201.93 53.34) (xy 205.74 53.34)
+		)
+		(stroke
+			(width 0)
+			(type default)
+		)
+	)
+	(global_label "USB_DP"
+		(shape output)
+		(at 205.74 53.34 0)
+		(fields_autoplaced yes)
+		(effects
+			(font
+				(size 1.27 1.27)
+			)
+			(justify left)
+		)
+		(property "Intersheetrefs" "${INTERSHEET_REFS}"
+			(at 216.0428 53.34 0)
+			(effects
+				(font
+					(size 1.27 1.27)
+				)
+				(justify left)
+				(hide yes)
+			)
+		)
+	)
+	(symbol
+		(lib_id "Device:R_Small")
+		(at 199.39 53.34 270)
+		(unit 1)
+		(exclude_from_sim no)
+		(in_bom yes)
+		(on_board yes)
+		(dnp no)
+		(property "Reference" "R12"
+			(at 198.374 56.134 90)
+			(effects
+				(font
+					(size 1.016 1.016)
+				)
+				(justify right)
+			)
+		)
+		(property "Value" "22"
+			(at 203.454 55.88 90)
+			(effects
+				(font
+					(size 1.27 1.27)
+				)
+				(justify right)
+			)
+		)
+		(property "Footprint" "Resistor_SMD:R_0603_1608Metric_Pad0.98x0.95mm_HandSolder"
+			(at 199.39 53.34 0)
+			(effects
+				(font
+					(size 1.27 1.27)
+				)
+				(hide yes)
+			)
+		)
+		(property "Datasheet" "~"
+			(at 199.39 53.34 0)
+			(effects
+				(font
+					(size 1.27 1.27)
+				)
+				(hide yes)
+			)
+		)
+		(property "Description" "Resistor, small symbol"
+			(at 199.39 53.34 0)
+			(effects
+				(font
+					(size 1.27 1.27)
+				)
+				(hide yes)
+			)
+		)
+		(pin "2"
+		)
+		(pin "1"
+		)
+		(instances
+			(project "CanaryCap"
+				(path "/406ad30e-b04c-4bb7-9588-aab8ab73084a"
+					(reference "R12")
+					(unit 1)
+				)
+			)
+		)
 	)
 	(sheet
