File: CanaryCap PCB/_autosave-CanaryCap.kicad_pcb (KiCad board)
At the start: 2 copper layers, 120 x 30 mm, 59 parts, among them J1 USB_C_Receptacle_USB2.0_16P, J2 Impact Connector, J3 Gas Connector, J4 Battery Connector, Q1 NMOS, Q2 PMOS_Substrate, SW1 SW_MEC_5E, SW2 SW_MEC_5E, SW3 SW_MEC_5E, U1 LMZM23601V5, U2 LM3940 3.3V-SOT223, U3 ESP32-C6FH4, U4 ADXL343

Commit message: Added todo
Parts:
- moved C3 27.4 mm to (140.4, -17.0)
- moved C4 11.5 mm to (149.9, -1.50)
- moved R4 0.50 mm to (157.4, -13.0)
Changed lines of the file:
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@@
 	(footprint "Capacitor_SMD:C_0603_1608Metric_Pad1.08x0.95mm_HandSolder"
 		(layer "F.Cu")
-		(at 154.783301 6.350299)
+		(at 140.3625 -17)
 		(descr "Capacitor SMD 0603 (1608 Metric), square (rectangular) end terminal, IPC-7351 nominal with elongated pad for handsoldering. (Body size source: IPC-SM-782 page 76, https://www.pcb-3d.com/wordpress/wp-content/uploads/ipc-sm-782a_amendment_1_and_2.pdf), generated with kicad-footprint-generator")
 		(tags "capacitor handsolder")
@@
 	(footprint "Capacitor_SMD:C_0603_1608Metric_Pad1.08x0.95mm_HandSolder"
 		(layer "F.Cu")
-		(at 154.783301 8.860299)
+		(at 149.8625 -1.5)
 		(descr "Capacitor SMD 0603 (1608 Metric), square (rectangular) end terminal, IPC-7351 nominal with elongated pad for handsoldering. (Body size source: IPC-SM-782 page 76, https://www.pcb-3d.com/wordpress/wp-content/uploads/ipc-sm-782a_amendment_1_and_2.pdf), generated with kicad-footprint-generator")
 		(tags "capacitor handsolder")
@@
 	(footprint "Resistor_SMD:R_0603_1608Metric_Pad0.98x0.95mm_HandSolder"
 		(layer "F.Cu")
-		(at 157.4125 -12.5)
+		(at 157.4125 -13)
 		(descr "Resistor SMD 0603 (1608 Metric), square (rectangular) end terminal, IPC-7351 nominal with elongated pad for handsoldering. (Body size source: IPC-SM-782 page 72, https://www.pcb-3d.com/wordpress/wp-content/uploads/ipc-sm-782a_amendment_1_and_2.pdf), generated with kicad-footprint-generator")
 		(tags "resistor handsolder")
