File: CanaryCap PCB/micro.kicad_sch (KiCad schematic)
At the start: 23 parts, among them SW1 SW_MEC_5E, SW2 SW_MEC_5E, SW3 SW_MEC_5E, U3 ESP32-C6FH4

Commit message: Added todo
Parts:
- renumbered C9 to C10, C10 to C11, C11 to C12, C12 to C13, C13 to C14, C14 to C15, C15 to C16, C16 to C17, C17 to C18, C18 to C19, C6 to C7, C7 to C8, C8 to C9, R1 to R3, R2 to R4, R3 to R5, R4 to R6
