File: CanaryCap PCB/micro.kicad_sch (KiCad schematic)
At the start: 22 parts, among them SW1 SW_MEC_5E, SW2 SW_MEC_5E, U1 ESP32-C6FH4

Commit message: Updated schematics for justin to work
Parts:
- renumbered C17 to C12, C16 to C13, C15 to C14, C14 to C15, C12 to C16, C6 to C17, C8 to C18, C7 to C19, C13 to C7, C19 to C8, R4 to R3, R5 to R4, R3 to R5, U1 to U3
Connections:
- net ANT_MICRO: now reaches U3.1 (ANT)
Other:
- moved on the sheet: C12, C13, C14, C15

Commit message: new changes
Parts:
- added SW3: SW_MEC_5E, Button_Switch_SMD:SW_SPST_EVQP2_MiddlePushTravel_H2.5mm, symbol Switch:SW_Push
Connections:
- net GNDREF: now also SW3.1
- net GAS_IN: now reaches U3.10 (GPIO4/MTMS)
- net GAS_DIG_IN: now reaches U3.11 (GPIO5/MTDI)
- net Impact_IO: now reaches U3.18 (GPIO14)
- net Impact_CLK: now reaches U3.19 (GPIO15)
- net at U3.23 (SDIO_CMD/GPIO18): now also SW3.2
Other:
- note added: "IMPACT CANCEL BUTTON"
Changed lines of the file:
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@@
 		(comment 1 "Sebastian Arthur")
+	)
+	(text "IMPACT CANCEL BUTTON\n"
+		(exclude_from_sim no)
+		(at 223.012 87.63 0)
+		(effects
+			(font
+				(size 1.27 1.27)
+			)
+		)
 	)
 	(text "NP0/C0G Capacitor for high speed and accuracy"
@@
 	)
 	(junction
+		(at 208.28 99.06)
+		(diameter 0)
+		(color 0 0 0 0)
+	)
+	(junction
 		(at 236.22 40.64)
 		(diameter 0)
@@
 	(wire
 		(pts
+			(xy 208.28 88.9) (xy 208.28 99.06)
+		)
+		(stroke
+			(width 0)
+			(type default)
+		)
+	)
+	(wire
+		(pts
 			(xy 151.13 134.62) (xy 153.67 134.62)
 		)
@@
 	(wire
 		(pts
+			(xy 196.85 78.74) (xy 208.28 78.74)
+		)
+		(stroke
+			(width 0)
+			(type default)
+		)
+	)
+	(wire
+		(pts
 			(xy 153.67 137.16) (xy 153.67 151.13)
 		)
@@
 	(wire
 		(pts
-			(xy 196.85 99.06) (xy 199.39 99.06)
+			(xy 196.85 99.06) (xy 208.28 99.06)
 		)
 		(stroke
@@
 	(wire
 		(pts
-			(xy 199.39 99.06) (xy 199.39 100.33)
+			(xy 208.28 99.06) (xy 208.28 100.33)
 		)
 		(stroke
@@
 		)
 	)
+	(global_label "Impact_CLK"
+		(shape bidirectional)
+		(at 196.85 71.12 0)
+		(fields_autoplaced yes)
+		(effects
+			(font
+				(size 1.27 1.27)
+			)
+			(justify left)
+		)
+		(property "Intersheetrefs" "${INTERSHEET_REFS}"
+			(at 211.8926 71.12 0)
+			(effects
+				(font
+					(size 1.27 1.27)
+				)
+				(justify left)
+				(hide yes)
+			)
+		)
+	)
+	(global_label "GAS_IN"
+		(shape input)
+		(at 140.97 78.74 180)
+		(fields_autoplaced yes)
+		(effects
+			(font
+				(size 1.27 1.27)
+			)
+			(justify right)
+		)
+		(property "Intersheetrefs" "${INTERSHEET_REFS}"
+			(at 131.5138 78.74 0)
+			(effects
+				(font
+					(size 1.27 1.27)
+				)
+				(justify right)
+				(hide yes)
+			)
+		)
+	)
+	(global_label "GAS_DIG_IN"
+		(shape input)
+		(at 140.97 81.28 180)
+		(fields_autoplaced yes)
+		(effects
+			(font
+				(size 1.27 1.27)
+			)
+			(justify right)
+		)
+		(property "Intersheetrefs" "${INTERSHEET_REFS}"
+			(at 127.4014 81.28 0)
+			(effects
+				(font
+					(size 1.27 1.27)
+				)
+				(justify right)
+				(hide yes)
+			)
+		)
+	)
 	(global_label "BOOT"
 		(shape output)
@@
 				)
 				(justify right)
+				(hide yes)
+			)
+		)
+	)
+	(global_label "Impact_IO"
+		(shape bidirectional)
+		(at 196.85 68.58 0)
+		(fields_autoplaced yes)
+		(effects
+			(font
+				(size 1.27 1.27)
+			)
+			(justify left)
+		)
+		(property "Intersheetrefs" "${INTERSHEET_REFS}"
+			(at 210.2598 68.58 0)
+			(effects
+				(font
+					(size 1.27 1.27)
+				)
+				(justify left)
 				(hide yes)
 			)
@@
 	)
 	(symbol
+		(lib_id "Switch:SW_Push")
+		(at 208.28 83.82 90)
+		(unit 1)
+		(exclude_from_sim no)
+		(in_bom yes)
+		(on_board yes)
+		(dnp no)
+		(property "Reference" "SW3"
+			(at 211.328 82.55 90)
+			(effects
+				(font
+					(size 1.27 1.27)
+				)
+				(justify right)
+			)
+		)
+		(property "Value" "SW_MEC_5E"
+			(at 211.328 85.09 90)
+			(effects
+				(font
+					(size 1.27 1.27)
+				)
+				(justify right)
+			)
+		)
+		(property "Footprint" "Button_Switch_SMD:SW_SPST_EVQP2_MiddlePushTravel_H2.5mm"
+			(at 203.2 83.82 0)
+			(effects
+				(font
+					(size 1.27 1.27)
+				)
+				(hide yes)
+			)
+		)
+		(property "Datasheet" "~"
+			(at 203.2 83.82 0)
+			(effects
+				(font
+					(size 1.27 1.27)
+				)
+				(hide yes)
+			)
+		)
+		(property "Description" "Push button switch, generic, two pins"
+			(at 208.28 83.82 0)
+			(effects
+				(font
+					(size 1.27 1.27)
+				)
+				(hide yes)
+			)
+		)
+		(pin "1"
+		)
+		(pin "2"
+		)
+		(instances
+			(project "CanaryCap"
+				(path "/406ad30e-b04c-4bb7-9588-aab8ab73084a/865b4f90-0093-4030-8a8d-928bbea99e0f"
+					(reference "SW3")
+					(unit 1)
+				)
+			)
+		)
+	)
+	(symbol
 		(lib_id "Device:R_Small")
 		(at 134.62 88.9 90)
@@
 	(symbol
 		(lib_id "power:GNDREF")
-		(at 199.39 100.33 0)
+		(at 208.28 100.33 0)
 		(unit 1)
 		(exclude_from_sim no)
@@
 		(fields_autoplaced yes)
 		(property "Reference" "#PWR018"
-			(at 199.39 106.68 0)
+			(at 208.28 106.68 0)
 			(effects
 				(font
@@
 		)
 		(property "Value" "GNDREF"
-			(at 199.39 105.41 0)
+			(at 208.28 105.41 0)
 			(effects
 				(font
@@
 		)
 		(property "Footprint" ""
-			(at 199.39 100.33 0)
+			(at 208.28 100.33 0)
 			(effects
 				(font
@@
 		)
 		(property "Datasheet" ""
-			(at 199.39 100.33 0)
+			(at 208.28 100.33 0)
 			(effects
 				(font
@@
 		)
 		(property "Description" "Power symbol creates a global label with name \"GNDREF\" , reference supply ground"
-			(at 199.39 100.33 0)
-			(effects
-				(font
+			(at 208.28 100.33 0)
+			(effects
+				(font

Commit message: FIXED IT MF
Parts:
- renumbered C11 to C10, C12 to C11, C13 to C12, C14 to C13, C15 to C14, C16 to C15, C17 to C16, C18 to C17, C19 to C18, C7 to C6, C8 to C7, C9 to C8, C10 to C9, R3 to R1, R4 to R2, R5 to R3, R6 to R4

Commit message: Finished level for packaging
Parts:
- removed SW3: SW_MEC_5E, Button_Switch_SMD:SW_SPST_EVQP2_MiddlePushTravel_H2.5mm, symbol Switch:SW_Push
- added C25: 1uF, Capacitor_SMD:C_0603_1608Metric_Pad1.08x0.95mm_HandSolder, symbol Device:C
- added D4, D5, D6, D7, D8: LED_Small, LED_SMD:LED_0603_1608Metric_Pad1.05x0.95mm_HandSolder, symbol Device:LED_Small
- added R15: 10k, Resistor_SMD:R_0603_1608Metric_Pad0.98x0.95mm_HandSolder, symbol Device:R_Small
- added R16, R17, R18, R19, R20: 100, Resistor_SMD:R_0603_1608Metric_Pad0.98x0.95mm_HandSolder, symbol Device:R_Small
- added SW4: SW_MEC_5E, Button_Switch_SMD:SW_SPST_EVQP2_MiddlePushTravel_H2.5mm, symbol Switch:SW_Push
Connections:
- net +3.3V: now also R15.1, R16.1
- net GNDREF: now also C25.2, D4.1 (K), D5.1 (K), D6.1 (K), D7.1 (K), D8.1 (K), SW4.1
- net HEARTBEAT: now reaches U3.23 (SDIO_CMD/GPIO18)
- net HEARTBEAT: now also R17.1
- net HEALTH: now reaches U3.24 (SDIO_CLK/GPIO19)
- net HEALTH: now also R18.1
- net STATUS: now reaches U3.25 (SDIO_DATA0/GPIO20)
- net STATUS: now also R19.1
- net PENDING: now reaches U3.26 (SDIO_DATA1/GPIO21)
- net PENDING: now also R20.1
- net CANCEL: now reaches U3.9 (GPIO3)
- net CANCEL: now also C25.1, R15.2, SW4.2
- new net: D5.2 (A), R17.2
- new net: D4.2 (A), R16.2
- new net: D6.2 (A), R18.2
- new net: D8.2 (A), R20.2
- new net: D7.2 (A), R19.2

Commit message: Me phinks I did it
Parts:
- added LS1: AT-1440-TT-R, AT-1440-TT-R:XDCR_AT-1440-TT-R, symbol AT-1440-TT-R:AT-1440-TT-R
Connections:
- net GNDREF: now also LS1.N
- net at U3.22 (U0RXD/GPIO17): now also LS1.P
Changed lines of the file:
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@@
 	(wire
 		(pts
+			(xy 246.38 76.2) (xy 246.38 82.55)
+		)
+		(stroke
+			(width 0)
+			(type default)
+		)
+	)
+	(wire
+		(pts
 			(xy 236.22 40.64) (xy 238.76 40.64)
 		)
@@
 	(wire
 		(pts
+			(xy 196.85 76.2) (xy 246.38 76.2)
+		)
+		(stroke
+			(width 0)
+			(type default)
+		)
+	)
+	(wire
+		(pts
 			(xy 218.44 60.96) (xy 218.44 58.42)
 		)
@@
 	)
 	(symbol
+		(lib_id "power:GNDREF")
+		(at 246.38 92.71 0)
+		(unit 1)
+		(exclude_from_sim no)
+		(in_bom yes)
+		(on_board yes)
+		(dnp no)
+		(fields_autoplaced yes)
+		(property "Reference" "#PWR039"
+			(at 246.38 99.06 0)
+			(effects
+				(font
+					(size 1.27 1.27)
+				)
+				(hide yes)
+			)
+		)
+		(property "Value" "GNDREF"
+			(at 246.38 97.79 0)
+			(effects
+				(font
+					(size 1.27 1.27)
+				)
+			)
+		)
+		(property "Footprint" ""
+			(at 246.38 92.71 0)
+			(effects
+				(font
+					(size 1.27 1.27)
+				)
+				(hide yes)
+			)
+		)
+		(property "Datasheet" ""
+			(at 246.38 92.71 0)
+			(effects
+				(font
+					(size 1.27 1.27)
+				)
+				(hide yes)
+			)
+		)
+		(property "Description" "Power symbol creates a global label with name \"GNDREF\" , reference supply ground"
+			(at 246.38 92.71 0)
+			(effects
+				(font
+					(size 1.27 1.27)
+				)
+				(hide yes)
+			)
+		)
+		(pin "1"
+		)
+		(instances
+			(project "CanaryCap"
+				(path "/406ad30e-b04c-4bb7-9588-aab8ab73084a/865b4f90-0093-4030-8a8d-928bbea99e0f"
+					(reference "#PWR039")
+					(unit 1)
+				)
+			)
+		)
+	)
+	(symbol
 		(lib_id "Switch:SW_Push")
 		(at 40.64 49.53 90)
@@
 					(unit 1)
 				)
+			)
+		)
+	)
+	(symbol
+		(lib_id "AT-1440-TT-R:AT-1440-TT-R")
+		(at 248.92 87.63 0)
+		(unit 1)
+		(exclude_from_sim no)
+		(in_bom yes)
+		(on_board yes)
+		(dnp no)
+		(fields_autoplaced yes)
+		(property "Reference" "LS1"
+			(at 252.73 86.5042 0)
+			(effects
+				(font
+					(size 1.27 1.27)
+				)
+				(justify left)
+			)
+		)
+		(property "Value" "AT-1440-TT-R"
+			(at 252.73 89.0442 0)
+			(effects
+				(font
+					(size 1.27 1.27)
+				)
+				(justify left)
+			)
+		)
+		(property "Footprint" "AT-1440-TT-R:XDCR_AT-1440-TT-R"
+			(at 248.92 87.63 0)
+			(effects
+				(font
+					(size 1.27 1.27)
+				)
+				(justify bottom)
+				(hide yes)
+			)
+		)
+		(property "Datasheet" ""
+			(at 248.92 87.63 0)
+			(effects
+				(font
+					(size 1.27 1.27)
+				)
+				(hide yes)
+			)
+		)
+		(property "Description" ""
+			(at 248.92 87.63 0)
+			(effects
+				(font
+					(size 1.27 1.27)
+				)
+				(hide yes)
+			)
+		)
+		(property "PARTREV" "2014/07/25"
+			(at 248.92 87.63 0)
+			(effects
+				(font
+					(size 1.27 1.27)
+				)
+				(justify bottom)
+				(hide yes)
+			)
+		)
+		(property "STANDARD" "Manufacturer Recommendations"
+			(at 248.92 87.63 0)
+			(effects
+				(font
+					(size 1.27 1.27)
+				)
+				(justify bottom)
+				(hide yes)
+			)
+		)
+		(property "MAXIMUM_PACKAGE_HEIGHT" "7.1 mm"
+			(at 248.92 87.63 0)
+			(effects
+				(font
+					(size 1.27 1.27)
+				)
+				(justify bottom)
+				(hide yes)
+			)
+		)
+		(property "MANUFACTURER" "PUI Audio"
+			(at 248.92 87.63 0)
+			(effects
+				(font
+					(size 1.27 1.27)
+				)
+				(justify bottom)
+				(hide yes)
+			)
+		)
+		(pin "P"
+		)
+		(pin "N"
+		)
+		(instances
+			(project ""
+				(path "/406ad30e-b04c-4bb7-9588-aab8ab73084a/865b4f90-0093-4030-8a8d-928bbea99e0f"
+					(reference "LS1")
+					(unit 1)
+				)

Commit message: YIPPEE
Parts:
- removed C10, C9: 10pF, Capacitor_SMD:C_0603_1608Metric_Pad1.08x0.95mm_HandSolder, symbol Device:C
- removed C11, C12, C15, C16: 0.1uF, Capacitor_SMD:C_0603_1608Metric_Pad1.08x0.95mm_HandSolder, symbol Device:C
- removed C13, C14, C18: 10uF, Capacitor_SMD:C_0603_1608Metric_Pad1.08x0.95mm_HandSolder, symbol Device:C
- removed C17: 1uF, Capacitor_SMD:C_0603_1608Metric_Pad1.08x0.95mm_HandSolder, symbol Device:C
- removed L1: 2nH, Inductor_SMD:L_0603_1608Metric, symbol Device:L
- removed LS1: AT-1440-TT-R, AT-1440-TT-R:XDCR_AT-1440-TT-R, symbol AT-1440-TT-R:AT-1440-TT-R
- removed R4: 5k, Resistor_SMD:R_0603_1608Metric_Pad0.98x0.95mm_HandSolder, symbol Device:R_Small
- removed U3: ESP32-C6FH4, Package_DFN_QFN:QFN-32-1EP_5x5mm_P0.5mm_EP3.7x3.7mm, symbol ESP-32-C6:ESP32-C6FH4
- removed XTAL1: FW4000044Q, CRYSTAL4_FW4000044Q_DIO, symbol ESP-32-C6:FW4000044Q
- added LS1: AT-1440-TT-R, Library:XDCR_AT-1440-TT-R, symbol ESP-32-C6:AT-1440-TT-R
- added U3: ESP32-C6-WROOM-1-N8, Library:XCVR_ESP32-C6-WROOM-1-N8, symbol ESP-32-C6:ESP32-C6-WROOM-1-N8
Connections:
- net +3.3V: now also U3.2 (3V3)
- net BOOT: now also U3.10 (IO8)
- net CANCEL: now also U3.23 (IO15)
- net GAS_DIG_IN: now also U3.11 (IO10)
- net GAS_IN: now also U3.12 (IO11)
- net GNDREF: now also LS1.N, U3.1 (GND), U3.28 (GND__1), U3.29_1 (GND__2), U3.29_2 (GND__3), U3.29_3 (GND__4), U3.29_4 (GND__5), U3.29_5 (GND__6), U3.29_6 (GND__7), U3.29_7 (GND__8), U3.29_8 (GND__9), U3.29_9 (GND__10)
- net HEALTH: now also U3.19 (IO21)
- net HEARTBEAT: now also U3.18 (IO20)
- net Impact_CLK: now also U3.9 (IO1)
- net Impact_IO: now also U3.8 (IO0)
- net PENDING: now also U3.21 (IO23)
- net STATUS: now also U3.20 (IO22)
- net USB_DN: now also U3.13 (IO12)
- net USB_DP: now also U3.14 (IO13)
- net at C8.1, R3.2: now also U3.3 (EN)
- new net BUZZER: LS1.P, U3.17 (IO19)
- new net TCK: U3.6 (IO6)
- new net TDI: U3.5 (IO5)
- new net TDO: U3.7 (IO7)
- new net TMS: U3.4 (IO4)
Other:
- note removed: "IMPACT CANCEL BUTTON"
- note removed: "NP0/C0G Capacitor for high speed and accuracy"
- note removed: "Please check to find a correct component here"
- moved on the sheet: C8, R3

Commit message: Capcb updates
Connections:
- net BUZZER: now also U3.16 (IO18); no longer U3.17 (IO19)
- net CANCEL: now also U3.21 (IO23); no longer U3.23 (IO15)
- net GAS_DIG_IN: now also U3.27 (IO2); no longer U3.11 (IO10)
- net GAS_IN: now also U3.26 (IO3); no longer U3.12 (IO11)
- net HEALTH: now also U3.18 (IO20); no longer U3.19 (IO21)
- net HEARTBEAT: now also U3.17 (IO19); no longer U3.18 (IO20)
- net Impact_CLK: now also U3.12 (IO11); no longer U3.9 (IO1)
- net Impact_IO: now also U3.11 (IO10); no longer U3.8 (IO0)
- net PENDING: now also U3.20 (IO22); no longer U3.21 (IO23)
- net STATUS: now also U3.19 (IO21); no longer U3.20 (IO22)
Changed lines of the file:
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@@
 	(global_label "BUZZER"
 		(shape output)
-		(at 190.5 62.23 0)
-		(fields_autoplaced yes)
-		(effects
-			(font
-				(size 1.27 1.27)
-			)
-			(justify left)
-		)
-		(property "Intersheetrefs" "${INTERSHEET_REFS}"
-			(at 200.9237 62.23 0)
+		(at 190.5 59.69 0)
+		(fields_autoplaced yes)
+		(effects
+			(font
+				(size 1.27 1.27)
+			)
+			(justify left)
+		)
+		(property "Intersheetrefs" "${INTERSHEET_REFS}"
+			(at 200.9237 59.69 0)
 			(effects
 				(font
@@
 	(global_label "PENDING"
 		(shape output)
-		(at 190.5 72.39 0)
-		(fields_autoplaced yes)
-		(effects
-			(font
-				(size 1.27 1.27)
-			)
-			(justify left)
-		)
-		(property "Intersheetrefs" "${INTERSHEET_REFS}"
-			(at 201.71 72.39 0)
+		(at 190.5 69.85 0)
+		(fields_autoplaced yes)
+		(effects
+			(font
+				(size 1.27 1.27)
+			)
+			(justify left)
+		)
+		(property "Intersheetrefs" "${INTERSHEET_REFS}"
+			(at 201.71 69.85 0)
 			(effects
 				(font
@@
 	(global_label "Impact_CLK"
 		(shape bidirectional)
-		(at 149.86 49.53 180)
-		(fields_autoplaced yes)
-		(effects
-			(font
-				(size 1.27 1.27)
-			)
-			(justify right)
-		)
-		(property "Intersheetrefs" "${INTERSHEET_REFS}"
-			(at 134.8174 49.53 0)
-			(effects
-				(font
-					(size 1.27 1.27)
-				)
-				(justify right)
+		(at 190.5 44.45 0)
+		(fields_autoplaced yes)
+		(effects
+			(font
+				(size 1.27 1.27)
+			)
+			(justify left)
+		)
+		(property "Intersheetrefs" "${INTERSHEET_REFS}"
+			(at 205.5426 44.45 0)
+			(effects
+				(font
+					(size 1.27 1.27)
+				)
+				(justify left)
 				(hide yes)
 			)
@@
 	(global_label "HEALTH"
 		(shape output)
-		(at 190.5 67.31 0)
-		(fields_autoplaced yes)
-		(effects
-			(font
-				(size 1.27 1.27)
-			)
-			(justify left)
-		)
-		(property "Intersheetrefs" "${INTERSHEET_REFS}"
-			(at 200.3795 67.31 0)
+		(at 190.5 64.77 0)
+		(fields_autoplaced yes)
+		(effects
+			(font
+				(size 1.27 1.27)
+			)
+			(justify left)
+		)
+		(property "Intersheetrefs" "${INTERSHEET_REFS}"
+			(at 200.3795 64.77 0)
 			(effects
 				(font
@@
 	(global_label "GAS_IN"
 		(shape input)
-		(at 190.5 44.45 0)
-		(fields_autoplaced yes)
-		(effects
-			(font
-				(size 1.27 1.27)
-			)
-			(justify left)
-		)
-		(property "Intersheetrefs" "${INTERSHEET_REFS}"
-			(at 199.9562 44.45 0)
-			(effects
-				(font
-					(size 1.27 1.27)
-				)
-				(justify left)
+		(at 149.86 54.61 180)
+		(fields_autoplaced yes)
+		(effects
+			(font
+				(size 1.27 1.27)
+			)
+			(justify right)
+		)
+		(property "Intersheetrefs" "${INTERSHEET_REFS}"
+			(at 140.4038 54.61 0)
+			(effects
+				(font
+					(size 1.27 1.27)
+				)
+				(justify right)
 				(hide yes)
 			)
@@
 	(global_label "GAS_DIG_IN"
 		(shape input)
-		(at 190.5 41.91 0)
-		(fields_autoplaced yes)
-		(effects
-			(font
-				(size 1.27 1.27)
-			)
-			(justify left)
-		)
-		(property "Intersheetrefs" "${INTERSHEET_REFS}"
-			(at 204.0686 41.91 0)
-			(effects
-				(font
-					(size 1.27 1.27)
-				)
-				(justify left)
+		(at 149.86 52.07 180)
+		(fields_autoplaced yes)
+		(effects
+			(font
+				(size 1.27 1.27)
+			)
+			(justify right)
+		)
+		(property "Intersheetrefs" "${INTERSHEET_REFS}"
+			(at 136.2914 52.07 0)
+			(effects
+				(font
+					(size 1.27 1.27)
+				)
+				(justify right)
 				(hide yes)
 			)
@@
 	(global_label "CANCEL"
 		(shape input)
-		(at 190.5 52.07 0)
-		(fields_autoplaced yes)
-		(effects
-			(font
-				(size 1.27 1.27)
-			)
-			(justify left)
-		)
-		(property "Intersheetrefs" "${INTERSHEET_REFS}"
-			(at 200.6214 52.07 0)
+		(at 190.5 72.39 0)
+		(fields_autoplaced yes)
+		(effects
+			(font
+				(size 1.27 1.27)
+			)
+			(justify left)
+		)
+		(property "Intersheetrefs" "${INTERSHEET_REFS}"
+			(at 200.6214 72.39 0)
 			(effects
 				(font
@@
 	(global_label "Impact_IO"
 		(shape bidirectional)
-		(at 149.86 46.99 180)
-		(fields_autoplaced yes)
-		(effects
-			(font
-				(size 1.27 1.27)
-			)
-			(justify right)
-		)
-		(property "Intersheetrefs" "${INTERSHEET_REFS}"
-			(at 136.4502 46.99 0)
-			(effects
-				(font
-					(size 1.27 1.27)
-				)
-				(justify right)
+		(at 190.5 41.91 0)
+		(fields_autoplaced yes)
+		(effects
+			(font
+				(size 1.27 1.27)
+			)
+			(justify left)
+		)
+		(property "Intersheetrefs" "${INTERSHEET_REFS}"
+			(at 203.9098 41.91 0)
+			(effects
+				(font
+					(size 1.27 1.27)
+				)
+				(justify left)
 				(hide yes)
 			)
@@
 	(global_label "HEARTBEAT"
 		(shape output)
-		(at 190.5 64.77 0)
-		(fields_autoplaced yes)
-		(effects
-			(font
-				(size 1.27 1.27)
-			)
-			(justify left)
-		)
-		(property "Intersheetrefs" "${INTERSHEET_REFS}"
-			(at 203.7661 64.77 0)
+		(at 190.5 62.23 0)
+		(fields_autoplaced yes)
+		(effects
+			(font
+				(size 1.27 1.27)
+			)
+			(justify left)
+		)
+		(property "Intersheetrefs" "${INTERSHEET_REFS}"
+			(at 203.7661 62.23 0)
 			(effects
 				(font
@@
 	(global_label "STATUS"
 		(shape output)
-		(at 190.5 69.85 0)
-		(fields_autoplaced yes)
-		(effects
-			(font
-				(size 1.27 1.27)
-			)
-			(justify left)
-		)
-		(property "Intersheetrefs" "${INTERSHEET_REFS}"
-			(at 200.2585 69.85 0)
-			(effects
-				(font
+		(at 190.5 67.31 0)
+		(fields_autoplaced yes)
+		(effects
+			(font
+				(size 1.27 1.27)
+			)
+			(justify left)
+		)
+		(property "Intersheetrefs" "${INTERSHEET_REFS}"
+			(at 200.2585 67.31 0)
+			(effects
+				(font
